File: mtk/design/BallSensor_Economy/KeyBall.kicad_pcb (KiCad board)
At the start: 2 copper layers, 22 x 25 mm, 22 parts, among them J1 Conn_01x07_Male, P1 Conn_01x01_Male, U1 TPS73601DBV, U2 TXS0102DCU, U3 TXS0102DCU, U4 PMW3360DM-T2QU

Commit message: elecrow order
Parts:
- U1: value TPS73601DBV -> TLV75801PDBVR
Changed lines of the file:
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@@
     (descr "SOT, 5 Pin (https://www.jedec.org/sites/default/files/docs/Mo-178c.PDF variant AA), generated with kicad-footprint-generator ipc_gullwing_generator.py")
     (tags "SOT TO_SOT_SMD")
-    (property "Description" "58dB@(100Hz),37dB@(10kHz) 400mA 200mV@(400mA) Adjustable 1.2V~5.5V Positive 1 5.5V SOT-23-5  Linear Voltage Regulators (LDO) ROHS")
-    (property "LCSC" "C59200")
+    (property "Description" "SOT-23-5 Linear Voltage Regulators (LDO) ROHS")
+    (property "LCSC" "C2877852")
     (property "Sheetfile" "KeyBall.kicad_sch")
     (property "Sheetname" "")
@@
       (effects (font (size 1 1) (thickness 0.15)))
     )
-    (fp_text value "TPS73601DBV" (at 0 2.4) (layer "F.Fab") hide
+    (fp_text value "TLV75801PDBVR" (at 0 2.4) (layer "F.Fab") hide
       (effects (font (size 1 1) (thickness 0.15)))
     )
