File: mtk/design/BallSensor_Economy/KeyBall.kicad_sch (KiCad schematic)
At the start: 22 parts, among them J1 Conn_01x07_Male, U1 TPS73601DBV, U2 TXS0102DCU, U3 TXS0102DCU, U4 PMW3360DM-T2QU

Commit message: elecrow order
Parts:
- C3: value (none) -> 100nF; footprint (none) -> Capacitor_SMD:C_0402_1005Metric
- P1: value (none) -> Conn_01x01_Male; footprint (none) -> TestPoint:TestPoint_Pad_D1.0mm
- R1: value (none) -> 33k; footprint (none) -> Resistor_SMD:R_0402_1005Metric
- R2: value (none) -> 56k; footprint (none) -> Resistor_SMD:R_0402_1005Metric
- R4, R6: value (none) -> 10k; footprint (none) -> Resistor_SMD:R_0603_1608Metric
- U1: value TPS73601DBV -> (none); footprint Package_TO_SOT_SMD:SOT-23-5 -> (none); LCSC C59200 -> C2877852
Changed lines of the file:
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@@
       (effects (font (size 1.27 1.27)) (justify left))
     )
-    (property "Value" "" (id 1) (at 160.02 146.0499 0)
-      (effects (font (size 1.27 1.27)) (justify left))
-    )
-    (property "Footprint" "" (id 2) (at 167.64 137.16 0))
+    (property "Value" "100nF" (id 1) (at 160.02 146.0499 0)
+      (effects (font (size 1.27 1.27)) (justify left))
+    )
+    (property "Footprint" "Capacitor_SMD:C_0402_1005Metric" (id 2) (at 167.64 137.16 0))
     (property "Datasheet" "https://datasheet.lcsc.com/lcsc/1810191219_Samsung-Electro-Mechanics-CL05B104KO5NNNC_C1525.pdf" (id 3) (at 156.21 144.78 0)
       (effects (font (size 1.27 1.27)) hide)
@@
       (effects (font (size 1.27 1.27)) (justify left))
     )
-    (property "Value" "" (id 1) (at 242.57 140.9699 0)
-      (effects (font (size 1.27 1.27)) (justify left))
-    )
-    (property "Footprint" "" (id 2) (at 238.252 139.7 90)
+    (property "Value" "10k" (id 1) (at 242.57 140.9699 0)
+      (effects (font (size 1.27 1.27)) (justify left))
+    )
+    (property "Footprint" "Resistor_SMD:R_0603_1608Metric" (id 2) (at 238.252 139.7 90)
       (effects (font (size 1.27 1.27)) hide)
     )
@@
       (effects (font (size 1.27 1.27)) (justify left))
     )
-    (property "Value" "" (id 1) (at 144.78 146.0499 0)
-      (effects (font (size 1.27 1.27)) (justify left))
-    )
-    (property "Footprint" "" (id 2) (at 140.462 146.05 90)
+    (property "Value" "33k" (id 1) (at 144.78 146.0499 0)
+      (effects (font (size 1.27 1.27)) (justify left))
+    )
+    (property "Footprint" "Resistor_SMD:R_0402_1005Metric" (id 2) (at 140.462 146.05 90)
       (effects (font (size 1.27 1.27)) hide)
     )
@@
     (in_bom yes) (on_board yes) (fields_autoplaced)
     (property "Reference" "U1" (id 0) (at 120.65 129.54 0))
-    (property "Value" "TPS73601DBV" (id 1) (at 120.65 132.08 0))
-    (property "Footprint" "Package_TO_SOT_SMD:SOT-23-5" (id 2) (at 120.65 133.985 0)
+    (property "Value" "" (id 1) (at 120.65 132.08 0))
+    (property "Footprint" "" (id 2) (at 120.65 133.985 0)
       (effects (font (size 1.27 1.27) italic) hide)
     )
-    (property "Datasheet" "http://www.ti.com/cn/lit/gpn/tps736" (id 3) (at 120.65 143.51 0)
-      (effects (font (size 1.27 1.27)) hide)
-    )
-    (property "LCSC" "C59200" (id 4) (at 120.65 134.62 0))
-    (property "Description" "58dB@(100Hz),37dB@(10kHz) 400mA 200mV@(400mA) Adjustable 1.2V~5.5V Positive 1 5.5V SOT-23-5  Linear Voltage Regulators (LDO) ROHS" (id 5) (at 120.65 142.24 0)
+    (property "Datasheet" "https://www.ti.com/product/TLV758P" (id 3) (at 120.65 143.51 0)
+      (effects (font (size 1.27 1.27)) hide)
+    )
+    (property "LCSC" "C2877852" (id 4) (at 120.65 134.62 0))
+    (property "Description" "SOT-23-5 Linear Voltage Regulators (LDO) ROHS" (id 5) (at 120.65 142.24 0)
       (effects (font (size 1.27 1.27)) hide)
     )
@@
       (effects (font (size 1.27 1.27)) (justify left))
     )
-    (property "Value" "" (id 1) (at 144.78 158.7499 0)
-      (effects (font (size 1.27 1.27)) (justify left))
-    )
-    (property "Footprint" "" (id 2) (at 140.462 157.48 90)
+    (property "Value" "56k" (id 1) (at 144.78 158.7499 0)
+      (effects (font (size 1.27 1.27)) (justify left))
+    )
+    (property "Footprint" "Resistor_SMD:R_0402_1005Metric" (id 2) (at 140.462 157.48 90)
       (effects (font (size 1.27 1.27)) hide)
     )
@@
       (effects (font (size 1.27 1.27)) (justify left))
     )
-    (property "Value" "" (id 1) (at 250.19 210.8199 0)
-      (effects (font (size 1.27 1.27)) (justify left))
-    )
-    (property "Footprint" "" (id 2) (at 245.872 209.55 90)
+    (property "Value" "10k" (id 1) (at 250.19 210.8199 0)
+      (effects (font (size 1.27 1.27)) (justify left))
+    )
+    (property "Footprint" "Resistor_SMD:R_0603_1608Metric" (id 2) (at 245.872 209.55 90)
       (effects (font (size 1.27 1.27)) hide)
     )
@@
       (effects (font (size 1.27 1.27)) (justify left))
     )
-    (property "Value" "" (id 1) (at 341.63 97.1549 90)
-      (effects (font (size 1.27 1.27)) (justify left))
-    )
-    (property "Footprint" "" (id 2) (at 340.36 95.25 0)
+    (property "Value" "Conn_01x01_Male" (id 1) (at 341.63 97.1549 90)
+      (effects (font (size 1.27 1.27)) (justify left))
+    )
+    (property "Footprint" "TestPoint:TestPoint_Pad_D1.0mm" (id 2) (at 340.36 95.25 0)
       (effects (font (size 1.27 1.27)) hide)
     )
@@
     )
     (path "/7a94e9d9-69e4-4e6f-9e30-49e371776587"
-      (reference "U1") (unit 1) (value "TPS73601DBV") (footprint "Package_TO_SOT_SMD:SOT-23-5")
+      (reference "U1") (unit 1) (value "TLV75801PDBVR") (footprint "Package_TO_SOT_SMD:SOT-23-5")
     )
     (path "/59bf4a5f-1b55-47e8-bba5-6b49f0c2255c"
